Commit message: Fix PID config loading and robot body color

File: urdf/omni_robot_forsyde.xacro (robot description, xacro)
@@ -66,4 +66,8 @@
     </sensor>
   </gazebo>
+  <!-- Fix robot body color (original xacro references link_chassis which doesn't exist) -->
+  <gazebo reference="base_link">
+    <material>Gazebo/Orange</material>
+  </gazebo>
   <!-- ================================================================
        Planar Move plugin — omni-directional motion for simulation

Commit message: Fix omni robot launch: PID namespace, TF conflict, body color
- Remove ns="/robot" from rosparam load (yaml already has robot: key,
  double-namespace broke PID gain lookup)
- Remove static odom->base_link transform that conflicted with the
  planar_move plugin's dynamic transform, causing robot motion issues
- Add joint_state_publisher so robot_state_publisher gets wheel states
- Change base_link material to Gazebo/Grey

File: urdf/omni_robot_forsyde.xacro (robot description, xacro)
@@ -66,7 +66,7 @@
     </sensor>
   </gazebo>
-  <!-- Fix robot body color (original xacro references link_chassis which doesn't exist) -->
+  <!-- Fix robot body color -->
   <gazebo reference="base_link">
-    <material>Gazebo/Orange</material>
+    <material>Gazebo/Grey</material>
   </gazebo>
   <!-- ================================================================
