Commit message: Replace two_plate_s.dae with body.stl to fix Ogre crash
two_plate_s.dae triggers an AxisAlignedBox assertion in Ogre 1.9
(Ubuntu 20.04) causing gzclient to abort on startup. body.stl is
a simpler mesh that renders correctly.

File: rob_pkg/omni_robot/urdf/my_model.xacro (robot description, xacro)
@@ -242,5 +242,5 @@
 	<origin xyz="0 0 ${base_z}" rpy="0 0 3.14"/>
 	<geometry>
-        <mesh filename="package://rob_pkg/meshes/two_plate_s.dae" />
+        <mesh filename="package://rob_pkg/meshes/body.stl" />
       </geometry>
       <material name="red"/>
@@ -249,5 +249,5 @@
 	<origin xyz="0 0 ${base_z}" rpy="0 0 3.14"/>
       <geometry>
-        <mesh filename="package://rob_pkg/meshes/two_plate_s.dae"   />
+        <mesh filename="package://rob_pkg/meshes/body.stl" />
       </geometry>
     </collision>

Commit message: Replace base_link mesh with cylinder primitive to fix Ogre crash
Ogre 1.9 on Ubuntu 20.04 aborts with AxisAlignedBox assertion on
both two_plate_s.dae and body.stl under software rendering.
A cylinder primitive avoids the mesh loader entirely.

File: rob_pkg/omni_robot/urdf/my_model.xacro (robot description, xacro)
@@ -240,14 +240,14 @@
     </inertial>
 	<visual>
-	<origin xyz="0 0 ${base_z}" rpy="0 0 3.14"/>
-	<geometry>
-        <mesh filename="package://rob_pkg/meshes/body.stl" />
+	<origin xyz="0 0 ${base_z}" rpy="0 0 0"/>
+	<geometry>
+        <cylinder radius="${rob_scale}" length="${rob_scale*0.3}"/>
       </geometry>
       <material name="red"/>
     </visual>
-    <collision >
-	<origin xyz="0 0 ${base_z}" rpy="0 0 3.14"/>
+    <collision>
+	<origin xyz="0 0 ${base_z}" rpy="0 0 0"/>
       <geometry>
-        <mesh filename="package://rob_pkg/meshes/body.stl" />
+        <cylinder radius="${rob_scale}" length="${rob_scale*0.3}"/>
       </geometry>
     </collision>
